File: STM32H7S7L8H6H_Board.kicad_pcb (KiCad board)
At the start: 4 copper layers, 1 part, among them IC1 STM32H7S7L8H6H

Commit message: Update
Other:
- board outline added: 100 x 100 mm
Changed lines of the file:
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@@
+		)
+	)
+	(gr_line
+		(start 40 150)
+		(end 40 50)
+		(stroke
+			(width 0.05)
+			(type default)
+		)
+		(layer "Edge.Cuts")
+	)
+	(gr_line
+		(start 40 50)
+		(end 140 50)
+		(stroke
+			(width 0.05)
+			(type default)
+		)
+		(layer "Edge.Cuts")
+	)
+	(gr_line
+		(start 140 50)
+		(end 140 150)
+		(stroke
+			(width 0.05)
+			(type default)
+		)
+		(layer "Edge.Cuts")
+	)
+	(gr_line
+		(start 140 150)
+		(end 40 150)
+		(stroke
+			(width 0.05)
+			(type default)
+		)
+		(layer "Edge.Cuts")
+	)
+	(gr_text_box "Notes:\n\n- PCBWay 4 layer with 0.45/0.3 mm hole $30 (100x100)\n- Impedance matching 4 layers"
+		(start 212.965 44.23)
+		(end 306.175 117.67)
+		(layer "In2.Cu")
+		(effects
+			(font
+				(size 1.5 1.5)
+				(thickness 0.3)
+				(bold yes)
+			)
+			(justify left top)
+		)
+		(border yes)
+		(stroke
+			(width 0.2)
+			(type solid)
 		)
 	)
