File: STM32H7S7L8H6H_Board.kicad_sch (KiCad schematic)
At the start: 134 parts, among them IC1 STM32H7S7L8H6H, J1 LPUART1_Headers, J10 Power Select Jumpers, J11 Debug_Pins, J12 User Button Jumper, J13 USB_B_Micro, J14 USB_B_Micro, J15 Debug_Pins, J2 I2C1_Headers, J3 Power Pins, J4 Pin_Headers, J5 SPI1_Headers, J6 Power Select Jumpers, J7 Coin Battery Jumper, J8 BOOT0_Jumper, J9 BOOT0_Jumper, U1 STM32WL55CCU6, U3 LD1117S18TR_SOT223, U4 FT230XS, U5 USBLC6-2SC6, Y1 ABM3B-32.000MHZ-8-R30-B1U-T, Y2 Clock_ECS-327MVATX-7-CN-TR, Y3 Clock_ECS-327MVATX-7-CN-TR, Y4 Oscillator_ASE-50.000MHZ-L-R-T

Commit message: Update
Parts:
- added C74, C75, C76, C77, C78, C79, C80: 100n, symbol Device:C
- added IC2: SDRAM_IS42S16320F-6TL, Personal_Project:SDRAM_IS42S16320F-6TL, symbol Personal_Projects:SDRAM_IS42S16320F-6TL
Connections:
- net +3.3V: now also C74.1, C75.1, C76.1, C77.1, C78.1, C79.1, C80.1, IC2.1 (VDD_1), IC2.14 (VDD_2), IC2.27 (VDD_3), IC2.3 (VDDQ_1), IC2.43 (VDDQ_3), IC2.9 (VDDQ_2)
- net GND: now also C74.2, C75.2, C76.2, C77.2, C78.2, C79.2, C80.2, IC2.12 (VSSQ_2), IC2.28 (VSS_1), IC2.41 (VSS_2), IC2.46 (VSSQ_3), IC2.52 (VSSQ_4), IC2.54 (VSS_3), IC2.6 (VSSQ_1)
- new net FMC_A0: IC2.23 (A0)
- new net FMC_A1: IC2.24 (A1)
- new net FMC_A10: IC2.22 (A10)
- new net FMC_A11: IC2.35 (A11)
- new net FMC_A12: IC2.36 (A12)
- new net FMC_A2: IC2.25 (A2)
- new net FMC_A3: IC2.26 (A3)
- new net FMC_A4: IC2.29 (A4)
- new net FMC_A5: IC2.30 (A5)
- new net FMC_A6: IC2.31 (A6)
- new net FMC_A7: IC2.32 (A7)
- new net FMC_A8: IC2.33 (A8)
- new net FMC_A9: IC2.34 (A9)
- new net FMC_BA0: IC2.20 (BA0)
- new net FMC_BA1: IC2.21 (BA1)
- new net FMC_D0: IC2.2 (DQ0)
- new net FMC_D1: IC2.4 (DQ1)
- new net FMC_D10: IC2.45 (DQ10)
- new net FMC_D11: IC2.47 (DQ11)
- new net FMC_D12: IC2.48 (DQ12)
- new net FMC_D13: IC2.50 (DQ13)
- new net FMC_D14: IC2.51 (DQ14)
- new net FMC_D15: IC2.53 (DQ15)
- new net FMC_D2: IC2.5 (DQ2)
- new net FMC_D3: IC2.7 (DQ3)
- new net FMC_D4: IC2.8 (DQ4)
- new net FMC_D5: IC2.10 (DQ5)
- new net FMC_D6: IC2.11 (DQ6)
- new net FMC_D7: IC2.13 (DQ7)
- new net FMC_D8: IC2.42 (DQ8)
- new net FMC_D9: IC2.44 (DQ9)
- new net FMC_NBL0: IC2.15 (DQML)
- new net FMC_NBL1: IC2.39 (DQMH)
- new net FMC_SDCKE0: IC2.37 (CKE)
- new net FMC_SDNCAS: IC2.17 (~{CAS})
- new net FMC_SDNE0: IC2.19 (~{CS})
- new net FMC_SDNRAS: IC2.18 (~{RAS})
- new net FMC_SDNWE: IC2.16 (~{WE})
- no-connect marks 14 -> 15
Other:
- note added: "Only need FMC_NBL0 and FMC_NBL1 due to 16 bit data bus"
- note added: "Place close SDRAM One for each VDD in SDRAM"

Commit message: Update
Parts:
- removed Y3: Clock_ECS-327MVATX-7-CN-TR, Personal_Project:Clock_ECS327MVATX7CNTR, symbol Personal_Projects:Clock_ECS-327MVATX-7-CN-TR
- added OS1: Oscillator_ECS-327MVATX-3-CN-TR, Personal_Project:Oscillator_ECS327MVATX3CNTR, symbol Personal_Projects:Oscillator_ECS-327MVATX-3-CN-TR
Connections:
- net +3.3V: now also OS1.4 (VDD)
- net GND: now also OS1.2 (GND)
- net at R13.1: now also OS1.3 (OUTPUT)
Other:
- moved on the sheet: C52

Commit message: Update
Parts:
- removed C38, C39: 1u, Capacitor_SMD:C_0805_2012Metric_Pad1.18x1.45mm_HandSolder, symbol Device:C
- removed LDO2: LDO_TLV75733PDBVR, Personal_Project:LDO_SOT95P280X145-5N, symbol Personal_Projects:LDO_TLV75733PDBVR
- added C81: 4u7, Capacitor_SMD:C_0603_1608Metric_Pad1.08x0.95mm_HandSolder, symbol Device:C
- added C82, C83: 1u, Capacitor_SMD:C_0805_2012Metric_Pad1.18x1.45mm_HandSolder, symbol Device:C
- added D1: BZX84C4V3LT1G, Package_TO_SOT_SMD:SOT-23, symbol Diode:BZX84Cxx
- added D2: BZX84C6V2LT1G, Package_TO_SOT_SMD:SOT-23, symbol Diode:BZX84Cxx
- added J16: JST_XH_2.54_Plug, Personal_Project:Connector_Power2pin_SHDRRA2W80P0X250_1X2_740X1150X610P, symbol Personal_Projects:Connector_Power2pin_JST_XH_2.54_Plug
- added J17: Power_Selector_Jumper, Connector_PinHeader_2.54mm:PinHeader_2x03_P2.54mm_Vertical, symbol Connector_Generic:Conn_02x03_Odd_Even
- added J18: 3V_Selection_Header, Connector_PinHeader_2.54mm:PinHeader_1x03_P2.54mm_Vertical, symbol Connector_Generic:Conn_01x03
- added LDO3: LDO_TLV75733PDBVR, Personal_Project:LDO_SOT95P280X145-5N, symbol Personal_Projects:LDO_TLV75733PDBVR
- added Q1: MOSFET_SI2333DDS-T1-BE3, Personal_Project:MOSFET_ SI2333DDS_SOT_DS-T1-BE3_VIS, symbol Personal_Projects:MOSFET_SI2333DDS-T1-BE3
- added R18: 100k, Resistor_SMD:R_0603_1608Metric_Pad0.98x0.95mm_HandSolder, symbol Device:R
- added S1: Switch_WS-SLSU SMT Mini Slide, Personal_Project:Switch_WS-SLSU SMT Mini Slide, symbol Personal_Projects:Switch_WS-SLSU SMT Mini Slide
- added Z1: Diode_BZX84C6V2-7-F, Personal_Project:Diode_BZX84C6V2_SOT96P240X110-3N, symbol Personal_Projects:Diode_BZX84C6V2-7-F
Connections:
- net +3.3V: now also S1.2
- net GND: now also C81.2, C82.2, C83.2, D1.1 (A), D2.1 (A), J16.1 (POWER-), LDO3.2 (GND), R18.2
- net VBUS_5V: now also D2.3 (K), J17.5 (Pin_5)
- new net EXT_POWER+: J16.2 (POWER+), Q1.3 (D)
- new net EXT_POWER+_NOLDO: J17.2 (Pin_2), J18.1 (Pin_1)
- new net EXT_POWER+_PP: D1.3 (K), J17.1 (Pin_1), J17.3 (Pin_3), Q1.2 (S), Z1.3 (K)
- new net LDO1_IN: C82.1, J17.4 (Pin_4), J17.6 (Pin_6), LDO3.1 (IN), LDO3.3 (EN)
- new net LDO1_OUT_3V3: C83.1, J18.3 (Pin_3), LDO3.5 (OUT)
- new net MOSFET_GATE: Q1.1 (G), R18.1, Z1.1 (A)
- new net POWER_3V3: C81.1, J18.2 (Pin_2), S1.1
- no-connect marks 15 -> 20
Other:
- note added: "Input voltage range: 1.45V to 5.5V"
- note added: "ON/OFF Switch"
- note added: "Overvoltage protection for the PMOSFET VGS (VGS max is 8V)"
- note added: "Polarity Protection"

Commit message: update
Parts:
- added J19: I2C1_Headers, Connector_PinHeader_2.54mm:PinHeader_2x03_P2.54mm_Horizontal, symbol Connector_Generic:Conn_02x03_Odd_Even
- added J20: LPUART1_Headers, Connector_PinHeader_2.54mm:PinHeader_2x03_P2.54mm_Horizontal, symbol Connector_Generic:Conn_02x03_Odd_Even
- added J21: SPI1_Headers, Connector_PinHeader_2.54mm:PinHeader_2x03_P2.54mm_Horizontal, symbol Connector_Generic:Conn_02x03_Odd_Even
- added R19, R20, R21, R22, R23: 33R, Resistor_SMD:R_0805_2012Metric, symbol Device:R
Connections:
- net GND: now also J19.2 (Pin_2), J19.3 (Pin_3), J19.4 (Pin_4), J19.6 (Pin_6), J20.2 (Pin_2), J20.3 (Pin_3), J20.4 (Pin_4), J20.6 (Pin_6), J21.2 (Pin_2), J21.6 (Pin_6)
- net PA1_SPI1_SCK: now also R22.1
- net PA2_LPUART1_TX: now also R19.2
- net PA3_LPUART1_RX: now also R20.1
- net PB5_SPI1_MOSI: now also R23.2
- net PB7_I2C1_SDA: now also J19.1 (Pin_1)
- net PB8_I2C1_SCL: now also J19.5 (Pin_5)
- new net: J20.5 (Pin_5), R20.2
- new net: J21.4 (Pin_4), R23.1
- new net: J21.1 (Pin_1), R21.2
- new net: J21.5 (Pin_5), R22.2
- new net: J20.1 (Pin_1), R19.1
- new net PB4_SPI1_MISO: R21.1
Other:
- note added: "Chip Select pin on general pin header"
